File: config-spi.kicad_sch (KiCad schematic)
At the start: 39 parts

Commit message: Added EN pullup for TPS54561 to avoid disabling by touch
Parts:
- C43: value (none) -> C_100n_0402_6V3; footprint (none) -> ddr5-testboard-footprints:0402-cap
- C44: value (none) -> C_47u_0603; footprint (none) -> ddr5-testboard-footprints:0603-cap
- C45, C46: value (none) -> C_470n_0402; footprint (none) -> ddr5-testboard-footprints:0402-cap
- D4: value (none) -> TPD6E05U06; footprint (none) -> ddr5-testboard-footprints:TPD6E05U06
- D5, D6: renamed from D?; value (none) -> KP-1608CGCK; footprint (none) -> ddr5-testboard-footprints:LED_0603
- EMCCLK1, PUDC_B1: value (none) -> TP_SMD1MM; footprint (none) -> ddr5-testboard-footprints:Testpoint_smd_1mm
- J3: value (none) -> 0878311420; footprint (none) -> ddr5-testboard-footprints:PinHeader_2x7_P2mm_Drill1mm
- MODE1: value (none) -> 61300311121; footprint (none) -> ddr5-testboard-footprints:PinHeader_1x3_P2.54_Drill1.1mm
- PROG_B1: value (none) -> B3U-1000P; footprint (none) -> ddr5-testboard-footprints:Switch_Tactile_SMD_B3U-1000P
- Q1, Q2: renamed from Q?; value (none) -> BSS138APW; footprint (none) -> ddr5-testboard-footprints:SC70-3
- R35, R36, R37, R38, R39, R40, R48, R49, R50, R51, R55: value (none) -> R_0R_0402; footprint (none) -> ddr5-testboard-footprints:0402-res
- R41: value (none) -> R_2k2_0402; footprint (none) -> ddr5-testboard-footprints:0402-res
- R42, R43, R56, R57: value (none) -> R_100R_0402; footprint (none) -> ddr5-testboard-footprints:0402-res
- R44, R45, R52, R53: value (none) -> R_4k7_0402; footprint (none) -> ddr5-testboard-footprints:0402-res
- R46, R47: renamed from R?; value (none) -> R_330R_0402; footprint (none) -> ddr5-testboard-footprints:0402-res
- R54: value (none) -> R_330R_0402; footprint (none) -> ddr5-testboard-footprints:0402-res
- U7: value (none) -> S25FL128SAGNFI000; footprint (none) -> ddr5-testboard-footprints:S25FL128SAGNFI000
- U8: value (none) -> XC7K160T-FFG676; footprint (none) -> ddr5-testboard-footprints:BGA676C100P26X26_2700X2700X254

Commit message: Update FPGA footprint reference
Parts:
- U8: footprint ddr5-testboard-footprints:BGA676C100P26X26_2700X2700X254 -> ddr5-testboard-footprints:xc7k160tfbg676
Changed lines of the file:
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@@
       (effects (font (size 1.27 1.27)) (justify right))
     )
-    (property "Footprint" "ddr5-testboard-footprints:BGA676C100P26X26_2700X2700X254" (id 2) (at 365.252 118.9736 0)
+    (property "Footprint" "ddr5-testboard-footprints:xc7k160tfbg676" (id 2) (at 365.252 118.9736 0)
       (effects (font (size 1.27 1.27)) (justify right) hide)
     )

Commit message: Update naming convention
Parts:
- C43: footprint ddr5-testboard-footprints:0402-cap -> data-center-rdimm-ddr5-tester-footprints:0402-cap; symbol ddr5-testboard:C_100n_0402_6V3 -> data-center-rdimm-ddr5-tester:C_100n_0402_6V3
- C44: footprint ddr5-testboard-footprints:0603-cap -> data-center-rdimm-ddr5-tester-footprints:0603-cap; symbol ddr5-testboard:C_47u_0603 -> data-center-rdimm-ddr5-tester:C_47u_0603
- C45, C46: footprint ddr5-testboard-footprints:0402-cap -> data-center-rdimm-ddr5-tester-footprints:0402-cap; symbol ddr5-testboard:C_470n_0402 -> data-center-rdimm-ddr5-tester:C_470n_0402
- D4: footprint ddr5-testboard-footprints:TPD6E05U06 -> data-center-rdimm-ddr5-tester-footprints:TPD6E05U06; symbol ddr5-testboard:TPD6E05U06 -> data-center-rdimm-ddr5-tester:TPD6E05U06
- D5, D6: footprint ddr5-testboard-footprints:LED_0603 -> data-center-rdimm-ddr5-tester-footprints:LED_0603; symbol ddr5-testboard:KP-1608CGCK -> data-center-rdimm-ddr5-tester:KP-1608CGCK
- EMCCLK1, PUDC_B1: footprint ddr5-testboard-footprints:Testpoint_smd_1mm -> data-center-rdimm-ddr5-tester-footprints:Testpoint_smd_1mm; symbol ddr5-testboard:TP_SMD1MM -> data-center-rdimm-ddr5-tester:TP_SMD1MM
- J3: footprint ddr5-testboard-footprints:PinHeader_2x7_P2mm_Drill1mm -> data-center-rdimm-ddr5-tester-footprints:PinHeader_2x7_P2mm_Drill1mm; symbol ddr5-testboard:0878311420 -> data-center-rdimm-ddr5-tester:0878311420
- MODE1: footprint ddr5-testboard-footprints:PinHeader_1x3_P2.54_Drill1.1mm -> data-center-rdimm-ddr5-tester-footprints:PinHeader_1x3_P2.54_Drill1.1mm; symbol ddr5-testboard:61300311121 -> data-center-rdimm-ddr5-tester:61300311121
- PROG_B1: footprint ddr5-testboard-footprints:Switch_Tactile_SMD_B3U-1000P -> data-center-rdimm-ddr5-tester-footprints:Switch_Tactile_SMD_B3U-1000P; symbol ddr5-testboard:B3U-1000P -> data-center-rdimm-ddr5-tester:B3U-1000P
- Q1, Q2: footprint ddr5-testboard-footprints:SC70-3 -> data-center-rdimm-ddr5-tester-footprints:SC70-3; symbol ddr5-testboard:BSS138APW -> data-center-rdimm-ddr5-tester:BSS138APW
- R35, R36, R37, R38, R39, R40, R48, R49, R50, R51, R55: footprint ddr5-testboard-footprints:0402-res -> data-center-rdimm-ddr5-tester-footprints:0402-res; symbol ddr5-testboard:R_0R_0402 -> data-center-rdimm-ddr5-tester:R_0R_0402
- R41: footprint ddr5-testboard-footprints:0402-res -> data-center-rdimm-ddr5-tester-footprints:0402-res; symbol ddr5-testboard:R_2k2_0402 -> data-center-rdimm-ddr5-tester:R_2k2_0402
- R42, R43, R56, R57: footprint ddr5-testboard-footprints:0402-res -> data-center-rdimm-ddr5-tester-footprints:0402-res; symbol ddr5-testboard:R_100R_0402 -> data-center-rdimm-ddr5-tester:R_100R_0402
- R44, R45, R52, R53: footprint ddr5-testboard-footprints:0402-res -> data-center-rdimm-ddr5-tester-footprints:0402-res; symbol ddr5-testboard:R_4k7_0402 -> data-center-rdimm-ddr5-tester:R_4k7_0402
- R46, R47, R54: footprint ddr5-testboard-footprints:0402-res -> data-center-rdimm-ddr5-tester-footprints:0402-res; symbol ddr5-testboard:R_330R_0402 -> data-center-rdimm-ddr5-tester:R_330R_0402
- U7: footprint ddr5-testboard-footprints:S25FL128SAGNFI000 -> data-center-rdimm-ddr5-tester-footprints:S25FL128SAGNFI000; symbol ddr5-testboard:S25FL128SAGNFI000 -> data-center-rdimm-ddr5-tester:S25FL128SAGNFI000
- U8: footprint ddr5-testboard-footprints:xc7k160tfbg676 -> data-center-rdimm-ddr5-tester-footprints:xc7k160tfbg676; symbol ddr5-testboard:XC7K160T-FFG676 -> data-center-rdimm-ddr5-tester:XC7K160T-FFG676
Other:
- title: DDR5 Tester -> Data Center RDIMM DDR5 Tester

Commit message: Introduce component standarization
Parts:
- C43: value C_100n_0402_6V3 -> C_100n_6V3_0402; footprint data-center-rdimm-ddr5-tester-footprints:0402-cap -> data-center-rdimm-ddr5-tester-footprints:C_0402_1005Metric; symbol data-center-rdimm-ddr5-tester:C_100n_0402_6V3 -> data-center-rdimm-ddr5-tester:C_100n_6V3_0402; Author (none) -> Antmicro; License (none) -> Apache-2.0
- C44: footprint data-center-rdimm-ddr5-tester-footprints:0603-cap -> data-center-rdimm-ddr5-tester-footprints:C_0603_1608Metric; Author (none) -> Antmicro; License (none) -> Apache-2.0; Manufacturer MURATA -> Murata
- C45, C46: footprint data-center-rdimm-ddr5-tester-footprints:0402-cap -> data-center-rdimm-ddr5-tester-footprints:C_0402_1005Metric; Author (none) -> Antmicro; License (none) -> Apache-2.0
- D4: value TPD6E05U06 -> TPD6E05U06RVZR; footprint data-center-rdimm-ddr5-tester-footprints:TPD6E05U06 -> data-center-rdimm-ddr5-tester-footprints:USON-14_3.5X1.3X0.5mm_P0.5mm; symbol data-center-rdimm-ddr5-tester:TPD6E05U06 -> data-center-rdimm-ddr5-tester:TPD6E05U06RVZR; Author (none) -> Antmicro; License (none) -> Apache-2.0
- D5, D6: value KP-1608CGCK -> LED_G_0603_KP-1608CGCK; footprint data-center-rdimm-ddr5-tester-footprints:LED_0603 -> data-center-rdimm-ddr5-tester-footprints:LED_0603_1608Metric_G; symbol data-center-rdimm-ddr5-tester:KP-1608CGCK -> data-center-rdimm-ddr5-tester:LED_G_0603_KP-1608CGCK; Author (none) -> Antmicro; License (none) -> Apache-2.0; Manufacturer KINGBRIGHT -> Kingbright
- EMCCLK1, PUDC_B1: value TP_SMD1MM -> TP_1mm_SMD; symbol data-center-rdimm-ddr5-tester:TP_SMD1MM -> data-center-rdimm-ddr5-tester:TP_1mm_SMD; Author (none) -> Antmicro; License (none) -> Apache-2.0
- J3: value 0878311420 -> PinHeader_2x7_P2mm_Drill1mm_Shrouded; footprint data-center-rdimm-ddr5-tester-footprints:PinHeader_2x7_P2mm_Drill1mm -> data-center-rdimm-ddr5-tester-footprints:PinHeader_2x7_P2mm_Drill1mm_Shrouded; symbol data-center-rdimm-ddr5-tester:0878311420 -> data-center-rdimm-ddr5-tester:PinHeader_2x7_P2mm_Drill1mm_Shrouded; Author (none) -> Antmicro; License (none) -> Apache-2.0; MPN 0878311420 -> 0878321420
- MODE1: value 61300311121 -> PinHeader_1x3_P2.54mm_Drill1.1mm; symbol data-center-rdimm-ddr5-tester:61300311121 -> data-center-rdimm-ddr5-tester:PinHeader_1x3_P2.54mm_Drill1.1mm; Author (none) -> Antmicro; License (none) -> Apache-2.0; Manufacturer Wurth Electronics Inc. -> Würth Elektronik
- PROG_B1: value B3U-1000P -> SW_B3U-1000P; footprint data-center-rdimm-ddr5-tester-footprints:Switch_Tactile_SMD_B3U-1000P -> data-center-rdimm-ddr5-tester-footprints:SW_B3U-3000P; symbol data-center-rdimm-ddr5-tester:B3U-1000P -> data-center-rdimm-ddr5-tester:SW_B3U-1000P; Author (none) -> Antmicro; License (none) -> Apache-2.0; Manufacturer Omron Electronics Inc-EMC Div -> Omron Electronics
- Q1, Q2: value BSS138APW -> BSS138PW; symbol data-center-rdimm-ddr5-tester:BSS138APW -> data-center-rdimm-ddr5-tester:BSS138PW; Author (none) -> Antmicro; License (none) -> Apache-2.0; Manufacturer ON Semiconductor -> Nexperia
- R35, R36, R37, R38, R39, R40, R48, R49, R50, R51, R55: footprint data-center-rdimm-ddr5-tester-footprints:0402-res -> data-center-rdimm-ddr5-tester-footprints:R_0402_1005Metric; Author (none) -> Antmicro; Current (none) -> 1A; License (none) -> Apache-2.0; Manufacturer PANASONIC -> Panasonic
- R41: footprint data-center-rdimm-ddr5-tester-footprints:0402-res -> data-center-rdimm-ddr5-tester-footprints:R_0402_1005Metric; Author (none) -> Antmicro; License (none) -> Apache-2.0; MPN RC0402FR-072K2L -> CR0402-FX-2201GLF; Manufacturer YAGEO -> Bourns; Tolerance (none) -> 1%
- R42, R43, R56, R57: footprint data-center-rdimm-ddr5-tester-footprints:0402-res -> data-center-rdimm-ddr5-tester-footprints:R_0402_1005Metric; Author (none) -> Antmicro; License (none) -> Apache-2.0; Manufacturer BOURNS -> Bourns; Tolerance (none) -> 1%
- R44, R45, R52, R53: footprint data-center-rdimm-ddr5-tester-footprints:0402-res -> data-center-rdimm-ddr5-tester-footprints:R_0402_1005Metric; Author (none) -> Antmicro; License (none) -> Apache-2.0; MPN ERJ2GEJ472X -> CR0402-FX-4701GLF; Manufacturer PANASONIC_ELECTRONIC_COMPONENTS -> Bourns; Tolerance (none) -> 1%
- R46, R47, R54: footprint data-center-rdimm-ddr5-tester-footprints:0402-res -> data-center-rdimm-ddr5-tester-footprints:R_0402_1005Metric; Author (none) -> Antmicro; License (none) -> Apache-2.0; MPN MCMR04X3300FTL -> CR0402-FX-3300GLF; Manufacturer MULTICOMP -> Bourns; Tolerance (none) -> 1%
- U7: footprint data-center-rdimm-ddr5-tester-footprints:S25FL128SAGNFI000 -> data-center-rdimm-ddr5-tester-footprints:WSON-8_6x8x0.5mm_P1.27mm; Author (none) -> Antmicro; License (none) -> Apache-2.0
- U8: footprint data-center-rdimm-ddr5-tester-footprints:xc7k160tfbg676 -> data-center-rdimm-ddr5-tester-footprints:BGA-676_27x27mm_Layout26x26_P1X1mm; Author (none) -> Antmicro; License (none) -> Apache-2.0; MPN (none) -> XC7K160T-FFG676; Manufacturer (none) -> Xilinx
Connections:
- net 3V3_SYS: now also R41.1; no longer R41.2
- net FCS_B: now also R41.2; no longer R41.1
- net GND: now also U7.9 (EP)
- net TCK_JTAG: now also D4.2 (D1-)
- net TDI_JTAG: now also D4.7 (D3-)
- net TDO_JTAG: now also D4.6 (D3+)
- net TMS_JTAG: now also D4.1 (D1+)
- net at D4.11 (D2-): now also D4.4 (D2-)
- net at D4.12 (D2+): now also D4.3 (D2+)
- no-connect marks 2 -> 4
Other:
- moved on the sheet: C43, C44, C45, C46, EMCCLK1, J3, PUDC_B1, R35, R36, R37, R38, R39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

Commit message: [#55296] component update
Parts:
- EMCCLK1, PUDC_B1: footprint data-center-rdimm-ddr5-tester-footprints:Testpoint_smd_1mm -> antmicro-footprints:TP_SMD_1mm
- J3: MPN 0878321420 -> 0878311420
- MODE1: footprint data-center-rdimm-ddr5-tester-footprints:PinHeader_1x3_P2.54_Drill1.1mm -> data-center-rdimm-ddr5-tester-footprints:PinHeader_1x3_P2.54mm_Drill1.1mm; VSD_class (none) -> IO Header
- PROG_B1: footprint data-center-rdimm-ddr5-tester-footprints:SW_B3U-3000P -> antmicro-footprints:SW_B3U-1000P_SMD; symbol data-center-rdimm-ddr5-tester:SW_B3U-1000P -> data-center-rdimm-ddr5-tester:SW_B3U-1000P_SMD; Manufacturer Omron Electronics -> Omron
- R42, R43, R49, R50, R57: now not fitted; now left out of the parts list
- U8: Manufacturer Xilinx -> AMD-Xilinx
Connections:
- net GND: no longer U7.9 (EP)
Other:
- moved on the sheet: R35
