File: interfaces.kicad_sch (KiCad schematic)
At the start: 87 parts

Commit message: Added EN pullup for TPS54561 to avoid disabling by touch
Parts:
- C148, C149, C154, C156, C157, C158, C159, C160, C161, C162: value (none) -> C_100n_0402_6V3; footprint (none) -> ddr5-testboard-footprints:0402-cap
- C150, C152, C155: value (none) -> C_4u7_0402; footprint (none) -> ddr5-testboard-footprints:0402-cap
- C151, C153: value (none) -> C_18p_0402; footprint (none) -> ddr5-testboard-footprints:0402-cap
- C163: value (none) -> C_1u_0603; footprint (none) -> ddr5-testboard-footprints:0603-cap
- D10, D11, D7, D8, D9: value (none) -> KP-1608CGCK; footprint (none) -> ddr5-testboard-footprints:LED_0603
- D12: value (none) -> TPD2E009; footprint (none) -> ddr5-testboard-footprints:SOT-3
- FB5, FB6, FB8: value (none) -> BLM18AG601SN1D; footprint (none) -> ddr5-testboard-footprints:0603
- FB7: renamed from FB?; value (none) -> BLM18PG121SN1D; footprint (none) -> ddr5-testboard-footprints:0603-res
- IC3: value (none) -> TPD8S009DSMR; footprint (none) -> ddr5-testboard-footprints:R-PDSO-N15
- J5: value (none) -> 685119134923; footprint (none) -> ddr5-testboard-footprints:HDMI_A_Female_685119134923
- J6: value (none) -> WE_629105150521; footprint (none) -> ddr5-testboard-footprints:USB_Micro_B_Female_629105150521
- J7: value (none) -> 1140084168; footprint (none) -> ddr5-testboard-footprints:MicroSD_1140084168
- PROG_B2, PROG_B3, PROG_B4, PROG_B5: renamed from PROG_B?; value (none) -> B3U-1000P; footprint (none) -> ddr5-testboard-footprints:Switch_Tactile_SMD_B3U-1000P
- Q3, Q4, Q5, Q6, Q7: value (none) -> BSS138APW; footprint (none) -> ddr5-testboard-footprints:SC70-3
- R100, R88, R89, R90, R91, R92, R93, R94, R95, R96, R97, R98, R99: value (none) -> R_22R_0402; footprint (none) -> ddr5-testboard-footprints:0402-res
- R101, R102, R103, R104, R105: value (none) -> R_330R_0402; footprint (none) -> ddr5-testboard-footprints:0402-res
- R106, R107, R109, R111, R113, R116, R118: value (none) -> R_20k_0402; footprint (none) -> ddr5-testboard-footprints:0402-res
- R108, R110, R112, R115, R117, R119, R120, R121: value (none) -> R_0R_0402; footprint (none) -> ddr5-testboard-footprints:0402-res
- R114: value (none) -> R_220R_0402; footprint (none) -> ddr5-testboard-footprints:0402-res
- R82, R83, R84, R85: renamed from R?; value (none) -> R_4k7_0402; footprint (none) -> ddr5-testboard-footprints:0402-res
- R86: value (none) -> R_12k_0402; footprint (none) -> ddr5-testboard-footprints:0402-res
- R87: value (none) -> R_10k_0402; footprint (none) -> ddr5-testboard-footprints:0402-res
- TP10, TP5, TP6, TP7, TP8, TP9: value (none) -> TP_SMD1MM; footprint (none) -> ddr5-testboard-footprints:Testpoint_smd_1mm
- U10: value (none) -> FT4232HQ; footprint (none) -> ddr5-testboard-footprints:FT4232HQ
- Y2: value (none) -> ABM8G-12.000MHZ-18-D2Y-T; footprint (none) -> ddr5-testboard-footprints:KX-7

Commit message: Update naming convention
Parts:
- C148, C149, C154, C156, C157, C158, C159, C160, C161, C162: footprint ddr5-testboard-footprints:0402-cap -> data-center-rdimm-ddr5-tester-footprints:0402-cap; symbol ddr5-testboard:C_100n_0402_6V3 -> data-center-rdimm-ddr5-tester:C_100n_0402_6V3
- C150, C152, C155: footprint ddr5-testboard-footprints:0402-cap -> data-center-rdimm-ddr5-tester-footprints:0402-cap; symbol ddr5-testboard:C_4u7_0402 -> data-center-rdimm-ddr5-tester:C_4u7_0402
- C151, C153: footprint ddr5-testboard-footprints:0402-cap -> data-center-rdimm-ddr5-tester-footprints:0402-cap; symbol ddr5-testboard:C_18p_0402 -> data-center-rdimm-ddr5-tester:C_18p_0402
- C163: footprint ddr5-testboard-footprints:0603-cap -> data-center-rdimm-ddr5-tester-footprints:0603-cap; symbol ddr5-testboard:C_1u_0603 -> data-center-rdimm-ddr5-tester:C_1u_0603
- D10, D11, D7, D8, D9: footprint ddr5-testboard-footprints:LED_0603 -> data-center-rdimm-ddr5-tester-footprints:LED_0603; symbol ddr5-testboard:KP-1608CGCK -> data-center-rdimm-ddr5-tester:KP-1608CGCK
- D12: footprint ddr5-testboard-footprints:SOT-3 -> data-center-rdimm-ddr5-tester-footprints:SOT-3; symbol ddr5-testboard:TPD2E009 -> data-center-rdimm-ddr5-tester:TPD2E009
- FB5, FB6, FB8: footprint ddr5-testboard-footprints:0603 -> data-center-rdimm-ddr5-tester-footprints:0603; symbol ddr5-testboard:BLM18AG601SN1D -> data-center-rdimm-ddr5-tester:BLM18AG601SN1D
- FB7: footprint ddr5-testboard-footprints:0603-res -> data-center-rdimm-ddr5-tester-footprints:0603-res; symbol ddr5-testboard:BLM18PG121SN1D -> data-center-rdimm-ddr5-tester:BLM18PG121SN1D
- IC3: footprint ddr5-testboard-footprints:R-PDSO-N15 -> data-center-rdimm-ddr5-tester-footprints:R-PDSO-N15; symbol ddr5-testboard:TPD8S009DSMR -> data-center-rdimm-ddr5-tester:TPD8S009DSMR
- J5: footprint ddr5-testboard-footprints:HDMI_A_Female_685119134923 -> data-center-rdimm-ddr5-tester-footprints:HDMI_A_Female_685119134923; symbol ddr5-testboard:685119134923 -> data-center-rdimm-ddr5-tester:685119134923
- J6: footprint ddr5-testboard-footprints:USB_Micro_B_Female_629105150521 -> data-center-rdimm-ddr5-tester-footprints:USB_Micro_B_Female_629105150521; symbol ddr5-testboard:WE_629105150521 -> data-center-rdimm-ddr5-tester:WE_629105150521
- J7: footprint ddr5-testboard-footprints:MicroSD_1140084168 -> data-center-rdimm-ddr5-tester-footprints:MicroSD_1140084168; symbol ddr5-testboard:1140084168 -> data-center-rdimm-ddr5-tester:1140084168
- PROG_B2, PROG_B3, PROG_B4, PROG_B5: footprint ddr5-testboard-footprints:Switch_Tactile_SMD_B3U-1000P -> data-center-rdimm-ddr5-tester-footprints:Switch_Tactile_SMD_B3U-1000P; symbol ddr5-testboard:B3U-1000P -> data-center-rdimm-ddr5-tester:B3U-1000P
- Q3, Q4, Q5, Q6, Q7: footprint ddr5-testboard-footprints:SC70-3 -> data-center-rdimm-ddr5-tester-footprints:SC70-3; symbol ddr5-testboard:BSS138APW -> data-center-rdimm-ddr5-tester:BSS138APW
- R100, R88, R89, R90, R91, R92, R93, R94, R95, R96, R97, R98, R99: footprint ddr5-testboard-footprints:0402-res -> data-center-rdimm-ddr5-tester-footprints:0402-res; symbol ddr5-testboard:R_22R_0402 -> data-center-rdimm-ddr5-tester:R_22R_0402
- R101, R102, R103, R104, R105: footprint ddr5-testboard-footprints:0402-res -> data-center-rdimm-ddr5-tester-footprints:0402-res; symbol ddr5-testboard:R_330R_0402 -> data-center-rdimm-ddr5-tester:R_330R_0402
- R106, R107, R109, R111, R113, R116, R118: footprint ddr5-testboard-footprints:0402-res -> data-center-rdimm-ddr5-tester-footprints:0402-res; symbol ddr5-testboard:R_20k_0402 -> data-center-rdimm-ddr5-tester:R_20k_0402
- R108, R110, R112, R115, R117, R119, R120, R121: footprint ddr5-testboard-footprints:0402-res -> data-center-rdimm-ddr5-tester-footprints:0402-res; symbol ddr5-testboard:R_0R_0402 -> data-center-rdimm-ddr5-tester:R_0R_0402
- R114: footprint ddr5-testboard-footprints:0402-res -> data-center-rdimm-ddr5-tester-footprints:0402-res; symbol ddr5-testboard:R_220R_0402 -> data-center-rdimm-ddr5-tester:R_220R_0402
- R82, R83, R84, R85: footprint ddr5-testboard-footprints:0402-res -> data-center-rdimm-ddr5-tester-footprints:0402-res; symbol ddr5-testboard:R_4k7_0402 -> data-center-rdimm-ddr5-tester:R_4k7_0402
- R86: footprint ddr5-testboard-footprints:0402-res -> data-center-rdimm-ddr5-tester-footprints:0402-res; symbol ddr5-testboard:R_12k_0402 -> data-center-rdimm-ddr5-tester:R_12k_0402
- R87: footprint ddr5-testboard-footprints:0402-res -> data-center-rdimm-ddr5-tester-footprints:0402-res; symbol ddr5-testboard:R_10k_0402 -> data-center-rdimm-ddr5-tester:R_10k_0402
- TP10, TP5, TP6, TP7, TP8, TP9: footprint ddr5-testboard-footprints:Testpoint_smd_1mm -> data-center-rdimm-ddr5-tester-footprints:Testpoint_smd_1mm; symbol ddr5-testboard:TP_SMD1MM -> data-center-rdimm-ddr5-tester:TP_SMD1MM
- U10: footprint ddr5-testboard-footprints:FT4232HQ -> data-center-rdimm-ddr5-tester-footprints:FT4232HQ; symbol ddr5-testboard:FT4232HQ -> data-center-rdimm-ddr5-tester:FT4232HQ
- Y2: footprint ddr5-testboard-footprints:KX-7 -> data-center-rdimm-ddr5-tester-footprints:KX-7; symbol ddr5-testboard:ABM8G-12.000MHZ-18-D2Y-T -> data-center-rdimm-ddr5-tester:ABM8G-12.000MHZ-18-D2Y-T
Other:
- title: DDR5 Tester -> Data Center RDIMM DDR5 Tester

Commit message: Introduce component standarization
Parts:
- C148, C149, C154, C156, C157, C158, C159, C160, C161, C162: value C_100n_0402_6V3 -> C_100n_6V3_0402; footprint data-center-rdimm-ddr5-tester-footprints:0402-cap -> data-center-rdimm-ddr5-tester-footprints:C_0402_1005Metric; symbol data-center-rdimm-ddr5-tester:C_100n_0402_6V3 -> data-center-rdimm-ddr5-tester:C_100n_6V3_0402; Author (none) -> Antmicro; License (none) -> Apache-2.0
- C150, C152, C155: footprint data-center-rdimm-ddr5-tester-footprints:0402-cap -> data-center-rdimm-ddr5-tester-footprints:C_0402_1005Metric; Author (none) -> Antmicro; License (none) -> Apache-2.0; Manufacturer MURATA -> Murata
- C151, C153: footprint data-center-rdimm-ddr5-tester-footprints:0402-cap -> data-center-rdimm-ddr5-tester-footprints:C_0402_1005Metric; Author (none) -> Antmicro; License (none) -> Apache-2.0; Manufacturer MULTICOMP -> Multicomp
- C163: footprint data-center-rdimm-ddr5-tester-footprints:0603-cap -> data-center-rdimm-ddr5-tester-footprints:C_0603_1608Metric; Author (none) -> Antmicro; License (none) -> Apache-2.0; Manufacturer WALSIN -> Walsin
- D10, D11, D7, D8, D9: value KP-1608CGCK -> LED_G_0603_KP-1608CGCK; footprint data-center-rdimm-ddr5-tester-footprints:LED_0603 -> data-center-rdimm-ddr5-tester-footprints:LED_0603_1608Metric_G; symbol data-center-rdimm-ddr5-tester:KP-1608CGCK -> data-center-rdimm-ddr5-tester:LED_G_0603_KP-1608CGCK; Author (none) -> Antmicro; License (none) -> Apache-2.0; Manufacturer KINGBRIGHT -> Kingbright
- D12: value TPD2E009 -> TPD2E009_SOT-9X3; footprint data-center-rdimm-ddr5-tester-footprints:SOT-3 -> data-center-rdimm-ddr5-tester-footprints:SOT-723; symbol data-center-rdimm-ddr5-tester:TPD2E009 -> data-center-rdimm-ddr5-tester:TPD2E009_SOT-9X3; Author (none) -> Antmicro; License (none) -> Apache-2.0
- FB5, FB6, FB8: value BLM18AG601SN1D -> FB_600Z_0.5A_0603; footprint data-center-rdimm-ddr5-tester-footprints:0603 -> data-center-rdimm-ddr5-tester-footprints:FB_0603_1608Metric; symbol data-center-rdimm-ddr5-tester:BLM18AG601SN1D -> data-center-rdimm-ddr5-tester:FB_600Z_0.5A_0603; Author (none) -> Antmicro; License (none) -> Apache-2.0; Manufacturer Murata Electronics North America -> Murata
- FB7: value BLM18PG121SN1D -> FB_120Z_2A_0603; footprint data-center-rdimm-ddr5-tester-footprints:0603-res -> data-center-rdimm-ddr5-tester-footprints:FB_0603_1608Metric; symbol data-center-rdimm-ddr5-tester:BLM18PG121SN1D -> data-center-rdimm-ddr5-tester:FB_120Z_2A_0603; Author (none) -> Antmicro; License (none) -> Apache-2.0; Manufacturer Murata Electronics North America -> Murata
- IC3: Author (none) -> Antmicro; License (none) -> Apache-2.0
- J5: value 685119134923 -> HDMI-A_685119134923; footprint data-center-rdimm-ddr5-tester-footprints:HDMI_A_Female_685119134923 -> data-center-rdimm-ddr5-tester-footprints:HDMI-A_Wurth_685119134923; symbol data-center-rdimm-ddr5-tester:685119134923 -> data-center-rdimm-ddr5-tester:HDMI-A_685119134923; Author (none) -> Antmicro; License (none) -> Apache-2.0; Manufacturer Amphenol -> Wurth Electronic
- J6: value WE_629105150521 -> USB_Micro-B_629105150521; symbol data-center-rdimm-ddr5-tester:WE_629105150521 -> data-center-rdimm-ddr5-tester:USB_Micro-B_629105150521; Author (none) -> Antmicro; License (none) -> Apache-2.0
- J7: value 1140084168 -> MicroSD_1140084168; footprint data-center-rdimm-ddr5-tester-footprints:MicroSD_1140084168 -> data-center-rdimm-ddr5-tester-footprints:MicroSD_Amphenol_1140084168; symbol data-center-rdimm-ddr5-tester:1140084168 -> data-center-rdimm-ddr5-tester:MicroSD_1140084168; Author (none) -> Antmicro; License (none) -> Apache-2.0
- PROG_B2, PROG_B3, PROG_B4, PROG_B5: value B3U-1000P -> SW_B3U-1000P; footprint data-center-rdimm-ddr5-tester-footprints:Switch_Tactile_SMD_B3U-1000P -> data-center-rdimm-ddr5-tester-footprints:SW_B3U-3000P; symbol data-center-rdimm-ddr5-tester:B3U-1000P -> data-center-rdimm-ddr5-tester:SW_B3U-1000P; Author (none) -> Antmicro; License (none) -> Apache-2.0; Manufacturer Omron Electronics Inc-EMC Div -> Omron Electronics
- Q3, Q4, Q5, Q6, Q7: value BSS138APW -> BSS138PW; symbol data-center-rdimm-ddr5-tester:BSS138APW -> data-center-rdimm-ddr5-tester:BSS138PW; Author (none) -> Antmicro; License (none) -> Apache-2.0; Manufacturer ON Semiconductor -> Nexperia
- R100, R88, R89, R90, R91, R92, R93, R94, R95, R96, R97, R98, R99: footprint data-center-rdimm-ddr5-tester-footprints:0402-res -> data-center-rdimm-ddr5-tester-footprints:R_0402_1005Metric; Author (none) -> Antmicro; License (none) -> Apache-2.0; MPN CRCW040222R0FKED -> CR0402-FX-22R0GLF; Manufacturer VISHAY -> Bourns; Tolerance (none) -> 1%
- R101, R102, R103, R104, R105: footprint data-center-rdimm-ddr5-tester-footprints:0402-res -> data-center-rdimm-ddr5-tester-footprints:R_0402_1005Metric; Author (none) -> Antmicro; License (none) -> Apache-2.0; MPN MCMR04X3300FTL -> CR0402-FX-3300GLF; Manufacturer MULTICOMP -> Bourns; Tolerance (none) -> 1%
- R106, R107, R109, R111, R113, R116, R118: footprint data-center-rdimm-ddr5-tester-footprints:0402-res -> data-center-rdimm-ddr5-tester-footprints:R_0402_1005Metric; Author (none) -> Antmicro; License (none) -> Apache-2.0; MPN CRCW040220K0FKED -> CR0402-FX-2002GLF; Manufacturer VISHAY -> Bourns; Tolerance (none) -> 1%
- R108, R110, R112, R115, R117, R119, R120, R121: footprint data-center-rdimm-ddr5-tester-footprints:0402-res -> data-center-rdimm-ddr5-tester-footprints:R_0402_1005Metric; Author (none) -> Antmicro; Current (none) -> 1A; License (none) -> Apache-2.0; Manufacturer PANASONIC -> Panasonic
- R114: footprint data-center-rdimm-ddr5-tester-footprints:0402-res -> data-center-rdimm-ddr5-tester-footprints:R_0402_1005Metric; Author (none) -> Antmicro; License (none) -> Apache-2.0; MPN ERJ2GEJ221X -> CR0402-FX-2200GLF; Manufacturer Panasonic -> Bourns; Tolerance (none) -> 1%
- R82, R83, R84, R85: footprint data-center-rdimm-ddr5-tester-footprints:0402-res -> data-center-rdimm-ddr5-tester-footprints:R_0402_1005Metric; Author (none) -> Antmicro; License (none) -> Apache-2.0; MPN ERJ2GEJ472X -> CR0402-FX-4701GLF; Manufacturer PANASONIC_ELECTRONIC_COMPONENTS -> Bourns; Tolerance (none) -> 1%
- R86: footprint data-center-rdimm-ddr5-tester-footprints:0402-res -> data-center-rdimm-ddr5-tester-footprints:R_0402_1005Metric; Author (none) -> Antmicro; License (none) -> Apache-2.0; MPN CRCW040212K0FKEDHP -> CR0402-FX-1202GLF; Manufacturer VISHAY -> Bourns; Tolerance (none) -> 1%
- R87: footprint data-center-rdimm-ddr5-tester-footprints:0402-res -> data-center-rdimm-ddr5-tester-footprints:R_0402_1005Metric; Author (none) -> Antmicro; License (none) -> Apache-2.0; MPN CRCW040210K0FKEDHP -> CR0402-FX-1002GLF; Manufacturer VISHAY -> Bourns; Tolerance (none) -> 1%
- TP10, TP5, TP6, TP7, TP8, TP9: value TP_SMD1MM -> TP_1mm_SMD; symbol data-center-rdimm-ddr5-tester:TP_SMD1MM -> data-center-rdimm-ddr5-tester:TP_1mm_SMD; Author (none) -> Antmicro; License (none) -> Apache-2.0
- U10: value FT4232HQ -> FT4232H_QFN; footprint data-center-rdimm-ddr5-tester-footprints:FT4232HQ -> data-center-rdimm-ddr5-tester-footprints:QFN-64_1EP_9x9mm_P0.5mm; symbol data-center-rdimm-ddr5-tester:FT4232HQ -> data-center-rdimm-ddr5-tester:FT4232H_QFN; Author (none) -> Antmicro; License (none) -> Apache-2.0
- Y2: value ABM8G-12.000MHZ-18-D2Y-T -> Oscillator_SMD_12MHz_KX-7; footprint data-center-rdimm-ddr5-tester-footprints:KX-7 -> data-center-rdimm-ddr5-tester-footprints:Oscillator_SMD_Geyer_KX-7-4Pin_3.2x2.5mm; symbol data-center-rdimm-ddr5-tester:ABM8G-12.000MHZ-18-D2Y-T -> data-center-rdimm-ddr5-tester:Oscillator_SMD_12MHz_KX-7; Author (none) -> Antmicro; License (none) -> Apache-2.0; Val (none) -> 12MHz
Connections:
- net GND: now also J7.SH (Shell); no longer J7.~ (Shell)
- no-connect marks 7 -> 26
Other:
- moved on the sheet: C148, C149, C150, C151, C152, C153, C154, C155, C156, C157, C158, C159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

Commit message: [#55296] component update
Parts:
- FB7: symbol data-center-rdimm-ddr5-tester:FB_120Z_2A_0603 -> data-center-rdimm-ddr5-tester:FB_120Z_2A_Murata-BLM18PG_0603; Val (none) -> 120Z/2A
- J5: footprint data-center-rdimm-ddr5-tester-footprints:HDMI-A_Wurth_685119134923 -> antmicro-footprints:HDMI-A_Receptacle_WE_685119134923; symbol data-center-rdimm-ddr5-tester:HDMI-A_685119134923 -> data-center-rdimm-ddr5-tester:HDMI-A_WE_685119134923; Manufacturer Wurth Electronic -> Würth Elektronik
- J6: footprint data-center-rdimm-ddr5-tester-footprints:USB_Micro_B_Female_629105150521 -> data-center-rdimm-ddr5-tester-footprints:USB-Micro-B_Receptacle_WE_629105150521; symbol data-center-rdimm-ddr5-tester:USB_Micro-B_629105150521 -> data-center-rdimm-ddr5-tester:USB-Micro-B_WE_629105150521; Manufacturer Wurth_Elektronik -> Würth Elektronik
- PROG_B2, PROG_B3, PROG_B4, PROG_B5: footprint data-center-rdimm-ddr5-tester-footprints:SW_B3U-3000P -> antmicro-footprints:SW_B3U-1000P_SMD; symbol data-center-rdimm-ddr5-tester:SW_B3U-1000P -> data-center-rdimm-ddr5-tester:SW_B3U-1000P_SMD; Manufacturer Omron Electronics -> Omron
- TP10, TP5, TP6, TP7, TP8, TP9: footprint data-center-rdimm-ddr5-tester-footprints:Testpoint_smd_1mm -> antmicro-footprints:TP_SMD_1mm
- U10: footprint data-center-rdimm-ddr5-tester-footprints:QFN-64_1EP_9x9mm_P0.5mm -> data-center-rdimm-ddr5-tester-footprints:QFN-64-1EP_9x9mm_P0.5mm; Manufacturer FTDI -> FTDI Chip
Connections:
- net at FB8.2: now also J6.SH (SHIELD); no longer J6.6
Other:
- moved on the sheet: D12, FB8, TP10, TP6, TP7, TP8, TP9
