File: supply.kicad_sch (KiCad schematic)
At the start: 125 parts

Commit message: Added EN pullup for TPS54561 to avoid disabling by touch
Parts:
- added R143: (no value), symbol ddr5-testboard:R_243k_0402
- 1V0, 1V1, 1V8, 3V3, 5V0, GND1, PHY1, TP1, TP2, TP3, TP4, VIN1: value (none) -> TP_SMD1MM; footprint (none) -> ddr5-testboard-footprints:Testpoint_smd_1mm
- C1, C2, C3, C4, C5, C6: value (none) -> C_47u_16V_1206; footprint (none) -> ddr5-testboard-footprints:1206-cap
- C10, C12: value (none) -> C_47p_0402; footprint (none) -> ddr5-testboard-footprints:0402-cap
- C11, C9: value (none) -> C_10n_0402; footprint (none) -> ddr5-testboard-footprints:0402-cap
- C13, C14: value (none) -> C_100n_0402_6V3; footprint (none) -> ddr5-testboard-footprints:0402-cap
- C15, C16, C17, C18, C19, C20: value (none) -> C_47u_0603; footprint (none) -> ddr5-testboard-footprints:0603-cap
- C177, C178, C179, C180, C181: value (none) -> C_1u_0402; footprint (none) -> antmicro-footprints:0402-cap
- C21, C22: value (none) -> C_10u_0402; footprint (none) -> ddr5-testboard-footprints:0402-cap
- C23, C24, C25: renamed from C?; value (none) -> C_10u_0402; footprint (none) -> ddr5-testboard-footprints:0402-cap
- C26, C27, C28, C29, C30, C42: renamed from C?; value (none) -> C_100n_0402_6V3; footprint (none) -> ddr5-testboard-footprints:0402-cap
- C31, C32, C33, C34, C35, C36, C37, C38, C39, C40: value (none) -> C_22u_0402; footprint (none) -> antmicro-footprints:0402-res
- C41: value (none) -> C_10n_0603; footprint (none) -> ddr5-testboard-footprints:0603-cap
- C7, C8: value (none) -> C_4n7_0402; footprint (none) -> ddr5-testboard-footprints:0402-cap
- D1, D2, D3: value (none) -> PDS760-13; footprint (none) -> ddr5-testboard-footprints:PDS760-13
- F1, F2, F3, F4, F5, F6, F7: value (none) -> 1206L450SLWR; footprint (none) -> ddr5-testboard-footprints:1206-res
- IC1, IC2: value (none) -> TPS54561; footprint (none) -> ddr5-testboard-footprints:WSON-10_4x4
- J1: value (none) -> DC_SOCKET; footprint (none) -> ddr5-testboard-footprints:DC_SOCKET
- J2: value (none) -> 61300311121; footprint (none) -> ddr5-testboard-footprints:PinHeader_1x3_P2.54_Drill1.1mm
- L1, L2: value (none) -> WE_7447798720; footprint (none) -> ddr5-testboard-footprints:WE_7447798720
- L3, L5, L6, L7, L8: value (none) -> SRP0420-1R5K; footprint (none) -> antmicro-footprints:SRP4020
- POT1: value (none) -> TC33X-2-203E; footprint (none) -> ddr5-testboard-footprints:Trimpot_3.8mmx3.6mm_TC33X-2-103E
- PWR1: value (none) -> KP-1608CGCK; footprint (none) -> ddr5-testboard-footprints:LED_0603
- R1, R142, R16, R17, R18, R19, R20: renamed from R?; value (none) -> R_0R_0402; footprint (none) -> ddr5-testboard-footprints:0402-res
- R10: value (none) -> R_43k_0402; footprint (none) -> ddr5-testboard-footprints:0402-res
- R11: value (none) -> R_100k_1%_0402; footprint (none) -> ddr5-testboard-footprints:0402
- R12, R15: value (none) -> R_10k2_0402; footprint (none) -> ddr5-testboard-footprints:0402-res
- R13: value (none) -> R_49R9_0402; footprint (none) -> ddr5-testboard-footprints:0402-res
- R14: value (none) -> R_53k6_0402; footprint (none) -> ddr5-testboard-footprints:0402-res
- R141, R24, R28, R30, R32, R33, R34: value (none) -> R_10k_0402; footprint (none) -> ddr5-testboard-footprints:0402-res
- R2, R3: value (none) -> R_16k9_0402; footprint (none) -> ddr5-testboard-footprints:0402-res
- R21: value (none) -> R_1k5_0402; footprint (none) -> antmicro-footprints:0402-res
- R22: value (none) -> R_1k_0402; footprint (none) -> antmicro-footprints:0402-res
- R23: value (none) -> R_12k4_0402; footprint (none) -> antmicro-footprints:0402-res
- R25: value (none) -> R_7k5_0402; footprint (none) -> antmicro-footprints:0402-res
- R26: value (none) -> R_20k_0402; footprint (none) -> ddr5-testboard-footprints:0402-res
- R27: value (none) -> R_31k6_0402; footprint (none) -> antmicro-footprints:0402-res
- R29: value (none) -> R_4k99_0402; footprint (none) -> antmicro-footprints:0402-res
- R31: value (none) -> R_0R_0402; footprint (none) -> ddr5-testboard-footprints:0402-res
- R4, R5: value (none) -> R_243k_0402; footprint (none) -> ddr5-testboard-footprints:0402-res
- R6: value (none) -> R_0R_2010; footprint (none) -> ddr5-testboard-footprints:2010-res
- R7: value (none) -> R_330R_0402; footprint (none) -> ddr5-testboard-footprints:0402-res
- R8, R9: value (none) -> R_100k_0402; footprint (none) -> ddr5-testboard-footprints:0402-res
- S1: value (none) -> EG1218; footprint (none) -> ddr5-testboard-footprints:Switch_Slide_11.6x4mm_EG1218
- U1, U2, U3, U4, U5: value (none) -> AP62301WU-7; footprint (none) -> antmicro-footprints:TSOT23-6
- U6: value (none) -> LM3881MME_NOPB; footprint (none) -> ddr5-testboard-footprints:VSSOP8-Texas_Instruments-DGK0008A
Connections:
- net SYS_EN: now also R143.1
- net VIN: now also R143.2
Other:
- moved on the sheet: TP1

Commit message: Update project libraries
Parts:
- C177, C178, C179, C180, C181: footprint antmicro-footprints:0402-cap -> ddr5-testboard-footprints:0402-cap; symbol antmicroCapacitors0402:C_1u_0402 -> ddr5-testboard:C_1u_0402
- C31, C32, C33, C34, C35, C36, C37, C38, C39, C40: footprint antmicro-footprints:0402-res -> ddr5-testboard-footprints:0402-res; symbol antmicroCapacitors0402:C_22u_0402 -> ddr5-testboard:C_22u_0402
- L3, L5, L6, L7, L8: footprint antmicro-footprints:SRP4020 -> ddr5-testboard-footprints:SRP4020; symbol antmicroFixedInductors:SRP0420-1R5K -> ddr5-testboard:SRP0420-1R5K
- R143: value (none) -> R_243k_0402; footprint (none) -> ddr5-testboard-footprints:0402-res
- R21: footprint antmicro-footprints:0402-res -> ddr5-testboard-footprints:0402-res; symbol antmicroResistors0402:R_1k5_0402 -> ddr5-testboard:R_1k5_0402
- R22: footprint antmicro-footprints:0402-res -> ddr5-testboard-footprints:0402-res; symbol antmicroResistors0402:R_1k_0402 -> ddr5-testboard:R_1k_0402
- R23: footprint antmicro-footprints:0402-res -> ddr5-testboard-footprints:0402-res; symbol antmicroResistors0402:R_12k4_0402 -> ddr5-testboard:R_12k4_0402
- R25: footprint antmicro-footprints:0402-res -> ddr5-testboard-footprints:0402-res; symbol antmicroResistors0402:R_7k5_0402 -> ddr5-testboard:R_7k5_0402
- R27: footprint antmicro-footprints:0402-res -> ddr5-testboard-footprints:0402-res; symbol antmicroResistors0402:R_31k6_0402 -> ddr5-testboard:R_31k6_0402
- R29: footprint antmicro-footprints:0402-res -> ddr5-testboard-footprints:0402-res; symbol antmicroResistors0402:R_4k99_0402 -> ddr5-testboard:R_4k99_0402
- U1, U2, U3, U4, U5: footprint antmicro-footprints:TSOT23-6 -> ddr5-testboard-footprints:TSOT23-6; symbol antmicroDCDCConverters:AP62301WU-7 -> ddr5-testboard:AP62301WU-7

Commit message: Update naming convention
Parts:
- 1V0, 1V1, 1V8, 3V3, 5V0, GND1, PHY1, TP1, TP2, TP3, TP4, VIN1: footprint ddr5-testboard-footprints:Testpoint_smd_1mm -> data-center-rdimm-ddr5-tester-footprints:Testpoint_smd_1mm; symbol ddr5-testboard:TP_SMD1MM -> data-center-rdimm-ddr5-tester:TP_SMD1MM
- C1, C2, C3, C4, C5, C6: footprint ddr5-testboard-footprints:1206-cap -> data-center-rdimm-ddr5-tester-footprints:1206-cap; symbol ddr5-testboard:C_47u_16V_1206 -> data-center-rdimm-ddr5-tester:C_47u_16V_1206
- C10, C12: footprint ddr5-testboard-footprints:0402-cap -> data-center-rdimm-ddr5-tester-footprints:0402-cap; symbol ddr5-testboard:C_47p_0402 -> data-center-rdimm-ddr5-tester:C_47p_0402
- C11, C9: footprint ddr5-testboard-footprints:0402-cap -> data-center-rdimm-ddr5-tester-footprints:0402-cap; symbol ddr5-testboard:C_10n_0402 -> data-center-rdimm-ddr5-tester:C_10n_0402
- C13, C14: footprint ddr5-testboard-footprints:0402-cap -> data-center-rdimm-ddr5-tester-footprints:0402-cap; symbol ddr5-testboard:C_100n_0402_6V3 -> data-center-rdimm-ddr5-tester:C_100n_0402_6V3
- C15, C16, C17, C18, C19, C20: footprint ddr5-testboard-footprints:0603-cap -> data-center-rdimm-ddr5-tester-footprints:0603-cap; symbol ddr5-testboard:C_47u_0603 -> data-center-rdimm-ddr5-tester:C_47u_0603
- C177, C178, C179, C180, C181: footprint ddr5-testboard-footprints:0402-cap -> data-center-rdimm-ddr5-tester-footprints:0402-cap; symbol ddr5-testboard:C_1u_0402 -> data-center-rdimm-ddr5-tester:C_1u_0402
- C21, C22, C23, C24, C25: footprint ddr5-testboard-footprints:0402-cap -> data-center-rdimm-ddr5-tester-footprints:0402-cap; symbol ddr5-testboard:C_10u_0402 -> data-center-rdimm-ddr5-tester:C_10u_0402
- C26, C27, C28, C29, C30, C42: footprint ddr5-testboard-footprints:0402-cap -> data-center-rdimm-ddr5-tester-footprints:0402-cap; symbol ddr5-testboard:C_100n_0402_6V3-antmicroCapacitors0402 -> data-center-rdimm-ddr5-tester:C_100n_0402_6V3-antmicroCapacitors0402
- C31, C32, C33, C34, C35, C36, C37, C38, C39, C40: footprint ddr5-testboard-footprints:0402-res -> data-center-rdimm-ddr5-tester-footprints:0402-res; symbol ddr5-testboard:C_22u_0402 -> data-center-rdimm-ddr5-tester:C_22u_0402
- C41: footprint ddr5-testboard-footprints:0603-cap -> data-center-rdimm-ddr5-tester-footprints:0603-cap; symbol ddr5-testboard:C_10n_0603 -> data-center-rdimm-ddr5-tester:C_10n_0603
- C7, C8: footprint ddr5-testboard-footprints:0402-cap -> data-center-rdimm-ddr5-tester-footprints:0402-cap; symbol ddr5-testboard:C_4n7_0402 -> data-center-rdimm-ddr5-tester:C_4n7_0402
- D1, D2, D3: footprint ddr5-testboard-footprints:PDS760-13 -> data-center-rdimm-ddr5-tester-footprints:PDS760-13; symbol ddr5-testboard:PDS760-13 -> data-center-rdimm-ddr5-tester:PDS760-13
- F1, F2, F3, F4, F5, F6, F7: footprint ddr5-testboard-footprints:1206-res -> data-center-rdimm-ddr5-tester-footprints:1206-res; symbol ddr5-testboard:1206L450SLWR -> data-center-rdimm-ddr5-tester:1206L450SLWR
- IC1, IC2: footprint ddr5-testboard-footprints:WSON-10_4x4 -> data-center-rdimm-ddr5-tester-footprints:WSON-10_4x4; symbol ddr5-testboard:TPS54561 -> data-center-rdimm-ddr5-tester:TPS54561
- J1: footprint ddr5-testboard-footprints:DC_SOCKET -> data-center-rdimm-ddr5-tester-footprints:DC_SOCKET; symbol ddr5-testboard:DC_SOCKET -> data-center-rdimm-ddr5-tester:DC_SOCKET
- J2: footprint ddr5-testboard-footprints:PinHeader_1x3_P2.54_Drill1.1mm -> data-center-rdimm-ddr5-tester-footprints:PinHeader_1x3_P2.54_Drill1.1mm; symbol ddr5-testboard:61300311121 -> data-center-rdimm-ddr5-tester:61300311121
- L1, L2: footprint ddr5-testboard-footprints:WE_7447798720 -> data-center-rdimm-ddr5-tester-footprints:WE_7447798720; symbol ddr5-testboard:WE_7447798720 -> data-center-rdimm-ddr5-tester:WE_7447798720
- L3, L5, L6, L7, L8: footprint ddr5-testboard-footprints:SRP4020 -> data-center-rdimm-ddr5-tester-footprints:SRP4020; symbol ddr5-testboard:SRP0420-1R5K -> data-center-rdimm-ddr5-tester:SRP0420-1R5K
- POT1: footprint ddr5-testboard-footprints:Trimpot_3.8mmx3.6mm_TC33X-2-103E -> data-center-rdimm-ddr5-tester-footprints:Trimpot_3.8mmx3.6mm_TC33X-2-103E; symbol ddr5-testboard:TC33X-2-203E -> data-center-rdimm-ddr5-tester:TC33X-2-203E
- PWR1: footprint ddr5-testboard-footprints:LED_0603 -> data-center-rdimm-ddr5-tester-footprints:LED_0603; symbol ddr5-testboard:KP-1608CGCK -> data-center-rdimm-ddr5-tester:KP-1608CGCK
- R1, R142, R16, R17, R18, R19, R20, R31: footprint ddr5-testboard-footprints:0402-res -> data-center-rdimm-ddr5-tester-footprints:0402-res; symbol ddr5-testboard:R_0R_0402 -> data-center-rdimm-ddr5-tester:R_0R_0402
- R10: footprint ddr5-testboard-footprints:0402-res -> data-center-rdimm-ddr5-tester-footprints:0402-res; symbol ddr5-testboard:R_43k_0402 -> data-center-rdimm-ddr5-tester:R_43k_0402
- R11: footprint ddr5-testboard-footprints:0402 -> data-center-rdimm-ddr5-tester-footprints:0402; symbol ddr5-testboard:R_100k_1%_0402 -> data-center-rdimm-ddr5-tester:R_100k_1%_0402
- R12, R15: footprint ddr5-testboard-footprints:0402-res -> data-center-rdimm-ddr5-tester-footprints:0402-res; symbol ddr5-testboard:R_10k2_0402 -> data-center-rdimm-ddr5-tester:R_10k2_0402
- R13: footprint ddr5-testboard-footprints:0402-res -> data-center-rdimm-ddr5-tester-footprints:0402-res; symbol ddr5-testboard:R_49R9_0402 -> data-center-rdimm-ddr5-tester:R_49R9_0402
- R14: footprint ddr5-testboard-footprints:0402-res -> data-center-rdimm-ddr5-tester-footprints:0402-res; symbol ddr5-testboard:R_53k6_0402 -> data-center-rdimm-ddr5-tester:R_53k6_0402
- R141, R24, R28, R30, R32, R33, R34: footprint ddr5-testboard-footprints:0402-res -> data-center-rdimm-ddr5-tester-footprints:0402-res; symbol ddr5-testboard:R_10k_0402 -> data-center-rdimm-ddr5-tester:R_10k_0402
- R143, R4, R5: footprint ddr5-testboard-footprints:0402-res -> data-center-rdimm-ddr5-tester-footprints:0402-res; symbol ddr5-testboard:R_243k_0402 -> data-center-rdimm-ddr5-tester:R_243k_0402
- R2, R3: footprint ddr5-testboard-footprints:0402-res -> data-center-rdimm-ddr5-tester-footprints:0402-res; symbol ddr5-testboard:R_16k9_0402 -> data-center-rdimm-ddr5-tester:R_16k9_0402
- R21: footprint ddr5-testboard-footprints:0402-res -> data-center-rdimm-ddr5-tester-footprints:0402-res; symbol ddr5-testboard:R_1k5_0402 -> data-center-rdimm-ddr5-tester:R_1k5_0402
- R22: footprint ddr5-testboard-footprints:0402-res -> data-center-rdimm-ddr5-tester-footprints:0402-res; symbol ddr5-testboard:R_1k_0402 -> data-center-rdimm-ddr5-tester:R_1k_0402
- R23: footprint ddr5-testboard-footprints:0402-res -> data-center-rdimm-ddr5-tester-footprints:0402-res; symbol ddr5-testboard:R_12k4_0402 -> data-center-rdimm-ddr5-tester:R_12k4_0402
- R25: footprint ddr5-testboard-footprints:0402-res -> data-center-rdimm-ddr5-tester-footprints:0402-res; symbol ddr5-testboard:R_7k5_0402 -> data-center-rdimm-ddr5-tester:R_7k5_0402
- R26: footprint ddr5-testboard-footprints:0402-res -> data-center-rdimm-ddr5-tester-footprints:0402-res; symbol ddr5-testboard:R_20k_0402 -> data-center-rdimm-ddr5-tester:R_20k_0402
- R27: footprint ddr5-testboard-footprints:0402-res -> data-center-rdimm-ddr5-tester-footprints:0402-res; symbol ddr5-testboard:R_31k6_0402 -> data-center-rdimm-ddr5-tester:R_31k6_0402
- R29: footprint ddr5-testboard-footprints:0402-res -> data-center-rdimm-ddr5-tester-footprints:0402-res; symbol ddr5-testboard:R_4k99_0402 -> data-center-rdimm-ddr5-tester:R_4k99_0402
- R6: footprint ddr5-testboard-footprints:2010-res -> data-center-rdimm-ddr5-tester-footprints:2010-res; symbol ddr5-testboard:R_0R_2010 -> data-center-rdimm-ddr5-tester:R_0R_2010
- R7: footprint ddr5-testboard-footprints:0402-res -> data-center-rdimm-ddr5-tester-footprints:0402-res; symbol ddr5-testboard:R_330R_0402 -> data-center-rdimm-ddr5-tester:R_330R_0402
- R8, R9: footprint ddr5-testboard-footprints:0402-res -> data-center-rdimm-ddr5-tester-footprints:0402-res; symbol ddr5-testboard:R_100k_0402 -> data-center-rdimm-ddr5-tester:R_100k_0402
- S1: footprint ddr5-testboard-footprints:Switch_Slide_11.6x4mm_EG1218 -> data-center-rdimm-ddr5-tester-footprints:Switch_Slide_11.6x4mm_EG1218; symbol ddr5-testboard:EG1218 -> data-center-rdimm-ddr5-tester:EG1218
- U1, U2, U3, U4, U5: footprint ddr5-testboard-footprints:TSOT23-6 -> data-center-rdimm-ddr5-tester-footprints:TSOT23-6; symbol ddr5-testboard:AP62301WU-7 -> data-center-rdimm-ddr5-tester:AP62301WU-7
- U6: footprint ddr5-testboard-footprints:VSSOP8-Texas_Instruments-DGK0008A -> data-center-rdimm-ddr5-tester-footprints:VSSOP8-Texas_Instruments-DGK0008A; symbol ddr5-testboard:LM3881MME_NOPB -> data-center-rdimm-ddr5-tester:LM3881MME_NOPB
Other:
- title: DDR5 Tester -> Data Center RDIMM DDR5 Tester

Commit message: Introduce component standarization
Parts:
- 1V0, 1V1, 1V8, 3V3, 5V0, GND1, PHY1, TP1, TP2, TP3, TP4, VIN1: value TP_SMD1MM -> TP_1mm_SMD; symbol data-center-rdimm-ddr5-tester:TP_SMD1MM -> data-center-rdimm-ddr5-tester:TP_1mm_SMD; Author (none) -> Antmicro; License (none) -> Apache-2.0
- C1, C2, C3, C4, C5, C6: footprint data-center-rdimm-ddr5-tester-footprints:1206-cap -> data-center-rdimm-ddr5-tester-footprints:C_1206_3216Metric; Author (none) -> Antmicro; License (none) -> Apache-2.0
- C10, C12: footprint data-center-rdimm-ddr5-tester-footprints:0402-cap -> data-center-rdimm-ddr5-tester-footprints:C_0402_1005Metric; Author (none) -> Antmicro; Dielectric (none) -> C0G; License (none) -> Apache-2.0; MPN C0402C470J5GACTU -> GRM1555C1E470JA01D; Manufacturer KEMET -> Murata
- C11, C9: footprint data-center-rdimm-ddr5-tester-footprints:0402-cap -> data-center-rdimm-ddr5-tester-footprints:C_0402_1005Metric; Author (none) -> Antmicro; Dielectric (none) -> X7R; License (none) -> Apache-2.0; MPN 04025G103ZAT2A -> GRM155R71H103KA88D; Manufacturer AVX -> Murata; Voltage (none) -> 50V
- C13, C14: value C_100n_0402_6V3 -> C_100n_6V3_0402; footprint data-center-rdimm-ddr5-tester-footprints:0402-cap -> data-center-rdimm-ddr5-tester-footprints:C_0402_1005Metric; symbol data-center-rdimm-ddr5-tester:C_100n_0402_6V3 -> data-center-rdimm-ddr5-tester:C_100n_6V3_0402; Author (none) -> Antmicro; License (none) -> Apache-2.0
- C15, C16, C17, C18, C19, C20: footprint data-center-rdimm-ddr5-tester-footprints:0603-cap -> data-center-rdimm-ddr5-tester-footprints:C_0603_1608Metric; Author (none) -> Antmicro; License (none) -> Apache-2.0; Manufacturer MURATA -> Murata
- C177, C178, C179, C180, C181, C7, C8: footprint data-center-rdimm-ddr5-tester-footprints:0402-cap -> data-center-rdimm-ddr5-tester-footprints:C_0402_1005Metric; Author (none) -> Antmicro; License (none) -> Apache-2.0
- C21, C22, C23, C24, C25: footprint data-center-rdimm-ddr5-tester-footprints:0402-cap -> data-center-rdimm-ddr5-tester-footprints:C_0402_1005Metric; Author (none) -> Antmicro; License (none) -> Apache-2.0; MPN GRM155R60J106ME44D -> CC0402MRX5R5BB106; Manufacturer MURATA -> Yaego
- C26, C27, C28, C29, C30, C42: value C_100n_0402_6V3 -> C_100n_6V3_0402; footprint data-center-rdimm-ddr5-tester-footprints:0402-cap -> data-center-rdimm-ddr5-tester-footprints:C_0402_1005Metric; symbol data-center-rdimm-ddr5-tester:C_100n_0402_6V3-antmicroCapacitors0402 -> data-center-rdimm-ddr5-tester:C_100n_6V3_0402; Author (none) -> Antmicro; License (none) -> Apache-2.0
- C31, C32, C33, C34, C35, C36, C37, C38, C39, C40: footprint data-center-rdimm-ddr5-tester-footprints:0402-res -> data-center-rdimm-ddr5-tester-footprints:C_0402_1005Metric; Author (none) -> Antmicro; License (none) -> Apache-2.0
- C41: footprint data-center-rdimm-ddr5-tester-footprints:0603-cap -> data-center-rdimm-ddr5-tester-footprints:C_0603_1608Metric; Author (none) -> Antmicro; License (none) -> Apache-2.0
- D1, D2, D3: value PDS760-13 -> PDS760; footprint data-center-rdimm-ddr5-tester-footprints:PDS760-13 -> data-center-rdimm-ddr5-tester-footprints:PowerDI5; symbol data-center-rdimm-ddr5-tester:PDS760-13 -> data-center-rdimm-ddr5-tester:PDS760; Author (none) -> Antmicro; License (none) -> Apache-2.0; Manufacturer Diodes Inc. -> Diodes Incorporated
- F1, F2, F3, F4, F5, F6, F7: value 1206L450SLWR -> PTC_4.5A_1206; footprint data-center-rdimm-ddr5-tester-footprints:1206-res -> data-center-rdimm-ddr5-tester-footprints:F_1206_3216Metric; symbol data-center-rdimm-ddr5-tester:1206L450SLWR -> data-center-rdimm-ddr5-tester:PTC_4.5A_1206; Author (none) -> Antmicro; License (none) -> Apache-2.0; Manufacturer LITTELFUSE -> Littelfuse
- IC1, IC2: value TPS54561 -> TPS54561QDPRRQ1; symbol data-center-rdimm-ddr5-tester:TPS54561 -> data-center-rdimm-ddr5-tester:TPS54561QDPRRQ1; Author (none) -> Antmicro; License (none) -> Apache-2.0; MPN TPS54561-Q1 -> TPS54561QDPRRQ1; Manufacturer Texas Instrumets -> Texas Instruments
- J1: value DC_SOCKET -> BarrelJack_3167288; footprint data-center-rdimm-ddr5-tester-footprints:DC_SOCKET -> data-center-rdimm-ddr5-tester-footprints:BarrelJack_3167288_Horizontal; symbol data-center-rdimm-ddr5-tester:DC_SOCKET -> data-center-rdimm-ddr5-tester:BarrelJack_3167288; Author (none) -> Antmicro; License (none) -> Apache-2.0
- J2: value 61300311121 -> PinHeader_1x3_P2.54mm_Drill1.1mm; symbol data-center-rdimm-ddr5-tester:61300311121 -> data-center-rdimm-ddr5-tester:PinHeader_1x3_P2.54mm_Drill1.1mm; Author (none) -> Antmicro; License (none) -> Apache-2.0; Manufacturer Wurth Electronics Inc. -> Würth Elektronik
- L1, L2: value WE_7447798720 -> L_7u2_7.9A_WE-PDF; footprint data-center-rdimm-ddr5-tester-footprints:WE_7447798720 -> data-center-rdimm-ddr5-tester-footprints:L_WE-PDF; symbol data-center-rdimm-ddr5-tester:WE_7447798720 -> data-center-rdimm-ddr5-tester:L_7u2_7.9A_WE-PDF; Author (none) -> Antmicro; License (none) -> Apache-2.0; Manufacturer Wurth Elektronik -> Würth Elektronik; Size (none) -> 10.2x10.2; Val (none) -> 7u2/7.9A
- L3, L5, L6, L7, L8: value SRP0420-1R5K -> L_1u5_6A_1716; footprint data-center-rdimm-ddr5-tester-footprints:SRP4020 -> data-center-rdimm-ddr5-tester-footprints:L_1716_4441Metric; symbol data-center-rdimm-ddr5-tester:SRP0420-1R5K -> data-center-rdimm-ddr5-tester:L_1u5_6A_1716; Author (none) -> Antmicro; License (none) -> Apache-2.0; MPN SRP0420-R47K -> SRP0420-1R5K; Manufacturer BOURNS -> Bourns
- POT1: Author (none) -> Antmicro; License (none) -> Apache-2.0; Manufacturer Bourns Inc. -> Bourns
- PWR1: value KP-1608CGCK -> LED_G_0603_KP-1608CGCK; footprint data-center-rdimm-ddr5-tester-footprints:LED_0603 -> data-center-rdimm-ddr5-tester-footprints:LED_0603_1608Metric_G; symbol data-center-rdimm-ddr5-tester:KP-1608CGCK -> data-center-rdimm-ddr5-tester:LED_G_0603_KP-1608CGCK; Author (none) -> Antmicro; License (none) -> Apache-2.0; Manufacturer KINGBRIGHT -> Kingbright
- R1, R142, R16, R17, R18, R19, R20, R31: footprint data-center-rdimm-ddr5-tester-footprints:0402-res -> data-center-rdimm-ddr5-tester-footprints:R_0402_1005Metric; Author (none) -> Antmicro; Current (none) -> 1A; License (none) -> Apache-2.0; Manufacturer PANASONIC -> Panasonic
- R10: footprint data-center-rdimm-ddr5-tester-footprints:0402-res -> data-center-rdimm-ddr5-tester-footprints:R_0402_1005Metric; Author (none) -> Antmicro; License (none) -> Apache-2.0; MPN 0402WGF4302TCE -> CR0402-FX-4302GLF; Manufacturer ROYAL_OHM -> Bourns; Tolerance (none) -> 1%
- R11: value R_100k_1%_0402 -> R_100k_0402; footprint data-center-rdimm-ddr5-tester-footprints:0402 -> data-center-rdimm-ddr5-tester-footprints:R_0402_1005Metric; symbol data-center-rdimm-ddr5-tester:R_100k_1%_0402 -> data-center-rdimm-ddr5-tester:R_100k_0402; Author (none) -> Antmicro; License (none) -> Apache-2.0; MPN ERA-6AEB104V -> CR0402-FX-1003GLF; Manufacturer PANASONIC -> Bourns; Tolerance (none) -> 1%; Val 100k_1% -> 100k
- R12, R15: footprint data-center-rdimm-ddr5-tester-footprints:0402-res -> data-center-rdimm-ddr5-tester-footprints:R_0402_1005Metric; Author (none) -> Antmicro; License (none) -> Apache-2.0; MPN MCWR04X1022FTL -> CR0402-FX-1022GLF; Manufacturer MULTICOMP PRO -> Bourns; Tolerance (none) -> 1%
- R13: footprint data-center-rdimm-ddr5-tester-footprints:0402-res -> data-center-rdimm-ddr5-tester-footprints:R_0402_1005Metric; Author (none) -> Antmicro; License (none) -> Apache-2.0; MPN CRCW040249R9FKED -> CR0402-FX-49R9GLF; Manufacturer VISHAY -> Bourns; Tolerance (none) -> 1%
- R14: footprint data-center-rdimm-ddr5-tester-footprints:0402-res -> data-center-rdimm-ddr5-tester-footprints:R_0402_1005Metric; Author (none) -> Antmicro; License (none) -> Apache-2.0; MPN CPF0402B53K6E1_ -> CR0402-FX-5362GLF; Manufacturer TE_CONNECTIVITY -> Bourns; Tolerance (none) -> 1%
- R141, R24, R28, R30, R32, R33, R34: footprint data-center-rdimm-ddr5-tester-footprints:0402-res -> data-center-rdimm-ddr5-tester-footprints:R_0402_1005Metric; Author (none) -> Antmicro; License (none) -> Apache-2.0; MPN CRCW040210K0FKEDHP -> CR0402-FX-1002GLF; Manufacturer VISHAY -> Bourns; Tolerance (none) -> 1%
- R143, R4, R5: footprint data-center-rdimm-ddr5-tester-footprints:0402-res -> data-center-rdimm-ddr5-tester-footprints:R_0402_1005Metric; Author (none) -> Antmicro; License (none) -> Apache-2.0; MPN MCMR04X2433FTL -> CR0402-FX-2433GLF; Manufacturer MULTICOMP -> Bourns; Tolerance (none) -> 1%
- R2, R3: footprint data-center-rdimm-ddr5-tester-footprints:0402-res -> data-center-rdimm-ddr5-tester-footprints:R_0402_1005Metric; Author (none) -> Antmicro; License (none) -> Apache-2.0; MPN ERA2AEB1692X -> CR0402-FX-1692GLF; Manufacturer PANASONIC -> Bourns; Tolerance (none) -> 1%
- R21: footprint data-center-rdimm-ddr5-tester-footprints:0402-res -> data-center-rdimm-ddr5-tester-footprints:R_0402_1005Metric; Author (none) -> Antmicro; License (none) -> Apache-2.0; MPN MP000515 -> CR0402-FX-1501GLF; Manufacturer Multicomp Pro -> Bourns; Tolerance (none) -> 1%
- R22: footprint data-center-rdimm-ddr5-tester-footprints:0402-res -> data-center-rdimm-ddr5-tester-footprints:R_0402_1005Metric; Author (none) -> Antmicro; License (none) -> Apache-2.0; Manufacturer BOURNS -> Bourns; Tolerance (none) -> 1%
- R23: footprint data-center-rdimm-ddr5-tester-footprints:0402-res -> data-center-rdimm-ddr5-tester-footprints:R_0402_1005Metric; Author (none) -> Antmicro; License (none) -> Apache-2.0; MPN ERJ2RKF1242X -> CR0402-FX-1242GLF; Manufacturer PANASONIC_ELECTRONIC_COMPONENTS -> Bourns; Tolerance (none) -> 1%
- R25: footprint data-center-rdimm-ddr5-tester-footprints:0402-res -> data-center-rdimm-ddr5-tester-footprints:R_0402_1005Metric; Author (none) -> Antmicro; License (none) -> Apache-2.0; MPN RC0402FR-077K5L -> CR0402-FX-7501GLF; Manufacturer YAGEO -> Bourns; Tolerance (none) -> 1%
- R26: footprint data-center-rdimm-ddr5-tester-footprints:0402-res -> data-center-rdimm-ddr5-tester-footprints:R_0402_1005Metric; Author (none) -> Antmicro; License (none) -> Apache-2.0; MPN CRCW040220K0FKED -> CR0402-FX-2002GLF; Manufacturer VISHAY -> Bourns; Tolerance (none) -> 1%
- R27: footprint data-center-rdimm-ddr5-tester-footprints:0402-res -> data-center-rdimm-ddr5-tester-footprints:R_0402_1005Metric; Author (none) -> Antmicro; License (none) -> Apache-2.0; MPN CRCW040231K6FKEDC -> CR0402-FX-3162GLF; Manufacturer Vishay -> Bourns; Tolerance (none) -> 1%
- R29: footprint data-center-rdimm-ddr5-tester-footprints:0402-res -> data-center-rdimm-ddr5-tester-footprints:R_0402_1005Metric; Author (none) -> Antmicro; License (none) -> Apache-2.0; MPN MCMR04X4991FTL -> CR0402-FX-4991GLF; Manufacturer MULTICOMP -> Bourns; Tolerance (none) -> 1%
- R6: footprint data-center-rdimm-ddr5-tester-footprints:2010-res -> data-center-rdimm-ddr5-tester-footprints:R_2010_5025Metric; Author (none) -> Antmicro; DNP DNP -> (none); License (none) -> Apache-2.0; Manufacturer VISHAY -> Vishay; Val 0R -> 0R
- R7: footprint data-center-rdimm-ddr5-tester-footprints:0402-res -> data-center-rdimm-ddr5-tester-footprints:R_0402_1005Metric; Author (none) -> Antmicro; License (none) -> Apache-2.0; MPN MCMR04X3300FTL -> CR0402-FX-3300GLF; Manufacturer MULTICOMP -> Bourns; Tolerance (none) -> 1%
- R8, R9: footprint data-center-rdimm-ddr5-tester-footprints:0402-res -> data-center-rdimm-ddr5-tester-footprints:R_0402_1005Metric; Author (none) -> Antmicro; License (none) -> Apache-2.0; MPN CRCW0402100KFKEDHP -> CR0402-FX-1003GLF; Manufacturer VISHAY -> Bourns; Tolerance (none) -> 1%
- S1: value EG1218 -> SW_EG1218; footprint data-center-rdimm-ddr5-tester-footprints:Switch_Slide_11.6x4mm_EG1218 -> data-center-rdimm-ddr5-tester-footprints:SW_Slide_E-Switch_EG1218; symbol data-center-rdimm-ddr5-tester:EG1218 -> data-center-rdimm-ddr5-tester:SW_EG1218; Author (none) -> Antmicro; License (none) -> Apache-2.0
- U1, U2, U3, U4, U5: footprint data-center-rdimm-ddr5-tester-footprints:TSOT23-6 -> data-center-rdimm-ddr5-tester-footprints:AP62301WU-7-TSOT23-6; Author (none) -> Antmicro; License (none) -> Apache-2.0
- U6: footprint data-center-rdimm-ddr5-tester-footprints:VSSOP8-Texas_Instruments-DGK0008A -> data-center-rdimm-ddr5-tester-footprints:VSSOP-8_3x3mm_P0.65mm; Author (none) -> Antmicro; License (none) -> Apache-2.0
Connections:
- net GND: now also C11.1, C41.2; no longer C11.2, C41.1
- net at U6.5 (TADJ): now also C41.1; no longer C41.2
- net at IC2.1 (BOOT): now also C14.1; no longer C14.2
- net at IC2.4 (SS/TR): now also C11.2; no longer C11.1
- net at D3.C, IC2.9 (SW), L2.1: now also C14.2; no longer C14.1
- net at L5.1, U2.2 (SW): now also C26.2; no longer C26.1
- net at U2.6 (BST): now also C26.1; no longer C26.2
- net at IC1.1 (BOOT): now also C13.1; no longer C13.2
- net at D2.C, IC1.9 (SW), L1.1: now also C13.2; no longer C13.1
- net at L8.1, U3.2 (SW): now also C28.2; no longer C28.1
- net at U3.6 (BST): now also C28.1; no longer C28.2
- net at L7.1, U5.2 (SW): now also C30.2; no longer C30.1
- net at U5.6 (BST): now also C30.1; no longer C30.2
- net at L3.1, U1.2 (SW): now also C27.2; no longer C27.1
- net at U1.6 (BST): now also C27.1; no longer C27.2
- net at L6.1, U4.2 (SW): now also C29.2; no longer C29.1
- net at U4.6 (BST): now also C29.1; no longer C29.2
- no-connect marks 2 -> 3
Other:
- moved on the sheet: 1V0, 1V1, 1V8, 3V3, 5V0, C1, C10, C11, C12, C13, C14, C15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

Commit message: [#55296] component update
Parts:
- 1V0, 1V1, 1V8, 3V3, 5V0, GND1, PHY1, TP1, TP2, TP3, TP4, VIN1: footprint data-center-rdimm-ddr5-tester-footprints:Testpoint_smd_1mm -> antmicro-footprints:TP_SMD_1mm
- IC1, IC2: footprint data-center-rdimm-ddr5-tester-footprints:WSON-10_4x4 -> data-center-rdimm-ddr5-tester-footprints:WSON-10-1EP_4x4mm_P0.8mm_EP2.6x3mm
- J1: Manufacturer Multicomp -> Multicomp Pro
- J2: footprint data-center-rdimm-ddr5-tester-footprints:PinHeader_1x3_P2.54_Drill1.1mm -> data-center-rdimm-ddr5-tester-footprints:PinHeader_1x3_P2.54mm_Drill1.1mm; VSD_class (none) -> IO Header
- R142: now not fitted; now left out of the parts list
- U1, U2, U3, U4, U5: footprint data-center-rdimm-ddr5-tester-footprints:AP62301WU-7-TSOT23-6 -> antmicro-footprints:TSOT23-6; symbol data-center-rdimm-ddr5-tester:AP62301WU-7 -> data-center-rdimm-ddr5-tester:AP62301_TSOT
- U6: symbol data-center-rdimm-ddr5-tester:LM3881MME_NOPB -> data-center-rdimm-ddr5-tester:LM3881
Other:
- moved on the sheet: C177, C178, C179, C181, C21, C22, C23, C25, C26, C28, C29, C30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
